File: MoxiE_Control_board.kicad_pcb (KiCad board)
At the start: 4 copper layers, 65 x 56 mm, 189 parts, among them J101 Conn_01x01, J102 Conn_01x01, J1101 USB_C_Receptacle, J401 +Vbat, J402 Gnd, J403 A, J404 B, J405 C, J406 Conn_01x03, K101 SERVO, P101 CANBUS, P102 CTRL_SIGNALS, P103 Serial1/tim4, P104 I2C, P106 HALL/Encoder, P801 SWD_DEBUG, P901 I2C, Q401 Q_PNP_BCE, Q501 TPH2R608NH,L1Q, Q502 TPH2R608NH,L1Q, Q503 TPH2R608NH,L1Q, Q504 TPH2R608NH,L1Q, Q601 TPH2R608NH,L1Q, Q602 TPH2R608NH,L1Q, Q603 TPH2R608NH,L1Q, Q604 TPH2R608NH,L1Q, Q701 TPH2R608NH,L1Q, Q702 TPH2R608NH,L1Q, Q703 TPH2R608NH,L1Q, Q704 TPH2R608NH,L1Q, SW801 SW_Push, U201 MAX3051, U301 TPS561201, U401 DRV8353RSRGZT, U801 STM32F40X_LQFP64, X801 8MHz 10ppm, X802 8MHz 10ppm

Commit message: pre pin refactor/remap incremental commit
Parts:
- removed C813: 100n, pkl_dipol:C_0402
- removed X802: 8MHz 10ppm, pkl_misc:PRQC
- R804: value 10k -> 1k
- X801: footprint Oscillators:Oscillator_SMD_EuroQuartz_XO53-4pin_5.0x3.2mm -> Oscillators:Oscillator_SMD_EuroQuartz_XO32-4pin_3.2x2.5mm
- moved X801 1.15 mm to (122.0, 142.0)
